File: driver_test.kicad_pcb (KiCad board)
At the start: 2 copper layers, 29.5 x 33.9 mm, 38 parts, among them M1 Module-knock-0.2, M2 Module-knock-0.2, U1 A4988_STEPPER_MOTOR_DRIVER_CA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, U2 TLE9201SG

Commit message: initial5
Parts:
- moved OUT_KNOCK1 1.00 mm to (136.3, 84.0)
- moved OUT_KNOCK2 1.00 mm to (136.3, 80.2)
- moved IN_KNOCK1 0.83 mm to (121.5, 83.0)
- moved IN_KNOCK2 0.83 mm to (121.5, 79.2)
Routing:
- net Net-(M1-OUT_KNOCK): track 2.16 -> 3.28 mm
- net Net-(M2-OUT_KNOCK): track 2.16 -> 3.15 mm
- net Net-(IN_KNOCK2-Pin_1): track 2.17 -> 3.14 mm
- net Net-(IN_KNOCK1-Pin_1): track 2.16 -> 3.10 mm
- added copper zone on In1.Cu, net GND
- added copper zone on In2.Cu, net GND
Other:
- copper layers 2 -> 4

Commit message: initial2
Parts:
- M1, M2: moved to B.Cu
- moved C16 9.81 mm to (123.9, 85.0), turned to -90 degrees
- moved 5V_IN1 9.03 mm to (130.3, 83.2)
- moved C4 9.03 mm to (127.3, 83.7)
- moved R6 9.03 mm to (130.4, 85.2)
- moved R7 9.03 mm to (127.3, 85.2)
- moved M2 6.32 mm to (124.7, 78.4)
- moved M1 6.29 mm to (124.6, 74.7)
- moved C15 5.85 mm to (121.8, 85.0), turned to -90 degrees
- moved OUT_KNOCK2 4.90 mm to (136.5, 75.3)
- moved OUT_KNOCK1 4.90 mm to (136.5, 79.1)
- moved C20 3.55 mm to (119.7, 85.0), turned to -90 degrees
- moved IN_KNOCK1 2.94 mm to (122.0, 80.1)
- moved IN_KNOCK2 2.81 mm to (122.0, 76.4)
Routing:
- net GND: track 128.1 -> 186.5 mm, vias 60 -> 66
- net +12VA: track 32.5 -> 48.5 mm
- net +5V: track 13.8 -> 19.2 mm
- net /VREF: track 14.8 -> 17.9 mm
- net /OUT-: track 6.74 -> 5.08 mm, vias 0 -> 2
